Commit message: Climbing feet cut: the bottom plate's end removed, as on our robot
Only the climbing feet change, on both feet:
- mjcf/assets/foot__configuration_right.stl: the cut foot (same frame and units)
- its collision pieces: 51 convex pieces (CoACD 0.02, <= 64 vertices) instead of 24
- the feet's inertials (MJCF, URDF): the CAD's minus the removed part, 29.98 g -> 25.74 g

The walking model, the hands and every other part are unchanged.

Co-Authored-By: Claude Opus 5.5 <noreply@anthropic.com>

File: src/microban_model/urdf/robot_climb.urdf (robot description, URDF)
Before this commit: robot microban, 28 links, 27 joints
Links:
- link foot_climb: mass 0.0299799 -> 0.0257414
- link foot_climb_2: mass 0.0299799 -> 0.0257414
